File: rev.2-heat/esp23 i3 heat thermostat/Indicator LED.kicad_sch (KiCad schematic)
At the start: 2 parts

Commit message: initial layout for UX
Parts:
- D10: renamed from D?; footprint (none) -> LED_SMD:LED_0603_1608Metric
- R21: renamed from R?; footprint (none) -> Resistor_SMD:R_0603_1608Metric
Changed lines of the file:
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@@
   (symbol (lib_id "Device:LED") (at 119.38 78.74 180)
     (in_bom yes) (on_board yes) (fields_autoplaced)
-    (property "Reference" "D?" (id 0) (at 120.9675 72.6145 0))
+    (property "Reference" "D10" (id 0) (at 120.9675 72.6145 0))
     (property "Value" "LED" (id 1) (at 120.9675 75.3896 0))
-    (property "Footprint" "" (id 2) (at 119.38 78.74 0)
+    (property "Footprint" "LED_SMD:LED_0603_1608Metric" (id 2) (at 119.38 78.74 0)
       (effects (font (size 1.27 1.27)) hide)
     )
@@
   (symbol (lib_id "power:GND") (at 123.19 78.74 0)
     (in_bom yes) (on_board yes) (fields_autoplaced)
-    (property "Reference" "#PWR?" (id 0) (at 123.19 85.09 0)
+    (property "Reference" "#PWR050" (id 0) (at 123.19 85.09 0)
       (effects (font (size 1.27 1.27)) hide)
     )
@@
   (symbol (lib_id "Device:R") (at 111.76 78.74 90)
     (in_bom yes) (on_board yes) (fields_autoplaced)
-    (property "Reference" "R?" (id 0) (at 111.76 73.7575 90))
+    (property "Reference" "R21" (id 0) (at 111.76 73.7575 90))
     (property "Value" "2.2k" (id 1) (at 111.76 76.5326 90))
-    (property "Footprint" "" (id 2) (at 111.76 80.518 90)
+    (property "Footprint" "Resistor_SMD:R_0603_1608Metric" (id 2) (at 111.76 80.518 90)
       (effects (font (size 1.27 1.27)) hide)
     )

Commit message: layout attempt 1
Parts:
- renumbered D10 to D8, R21 to R19
Changed lines of the file:
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@@
   (symbol (lib_id "Device:LED") (at 119.38 78.74 180)
     (in_bom yes) (on_board yes) (fields_autoplaced)
-    (property "Reference" "D10" (id 0) (at 120.9675 72.6145 0))
+    (property "Reference" "D8" (id 0) (at 120.9675 72.6145 0))
     (property "Value" "LED" (id 1) (at 120.9675 75.3896 0))
     (property "Footprint" "LED_SMD:LED_0603_1608Metric" (id 2) (at 119.38 78.74 0)
@@
   (symbol (lib_id "power:GND") (at 123.19 78.74 0)
     (in_bom yes) (on_board yes) (fields_autoplaced)
-    (property "Reference" "#PWR050" (id 0) (at 123.19 85.09 0)
+    (property "Reference" "#PWR048" (id 0) (at 123.19 85.09 0)
       (effects (font (size 1.27 1.27)) hide)
     )
@@
   (symbol (lib_id "Device:R") (at 111.76 78.74 90)
     (in_bom yes) (on_board yes) (fields_autoplaced)
-    (property "Reference" "R21" (id 0) (at 111.76 73.7575 90))
+    (property "Reference" "R19" (id 0) (at 111.76 73.7575 90))
     (property "Value" "2.2k" (id 1) (at 111.76 76.5326 90))
     (property "Footprint" "Resistor_SMD:R_0603_1608Metric" (id 2) (at 111.76 80.518 90)
