File: rev.2-heat/esp23 i3 heat thermostat/esp23 i3 heat thermostat.kicad_sch (KiCad schematic)
At the start: 47 parts

Commit message: initial layout for UX
Parts:
- added LED7, LED8: LTS-6980HR, Display_7Segment:7SegmentLED_LTS6760_LTS6780, symbol Display_Character:LTS-6980HR
- J1: renamed from J?; footprint (none) -> Connector_Phoenix_MC:PhoenixContact_MC_1,5_6-G-3.5_1x06_P3.50mm_Horizontal
- gave numbers to parts that had none: 46
Connections:
- net A: now also LED7.7 (a), LED8.7 (a)
- net B: now also LED7.6 (b), LED8.6 (b)
- net C: now also LED7.4 (c), LED8.4 (c)
- net D: now also LED7.2 (d), LED8.2 (d)
- net D1: now also LED8.3 (C.K.), LED8.8 (C.K.)
- net D2: now also LED6.3 (C.K.), LED6.8 (C.K.)
- net D3: now also LED4.3 (C.K.), LED4.8 (C.K.); no longer LED6.3 (C.K.), LED6.8 (C.K.)
- net D4: now also LED2.3 (C.K.), LED2.8 (C.K.); no longer LED4.3 (C.K.), LED4.8 (C.K.)
- net D5: now also LED7.3 (C.K.), LED7.8 (C.K.); no longer LED2.3 (C.K.), LED2.8 (C.K.)
- net DP: now also LED7.5 (DP), LED8.5 (DP)
- net E: now also LED7.1 (e), LED8.1 (e)
- net F: now also LED7.9 (f), LED8.9 (f)
- net G: now also LED7.10 (g), LED8.10 (g)

Commit message: layout attempt 1
Parts:
- removed C2: 0.1uF, Capacitor_SMD:C_0603_1608Metric, symbol Device:C
- removed C4: 1nF, Capacitor_SMD:C_0603_1608Metric, symbol Device:C
- removed D1: heat, LED_SMD:LED_0603_1608Metric, symbol Device:LED
- removed D2: fan, LED_SMD:LED_0603_1608Metric, symbol Device:LED
- removed D7: RED LED, LED_SMD:LED_0603_1608Metric, symbol Device:LED
- removed J3: Conn_02x05_Odd_Even, Connector_PinHeader_2.54mm:PinHeader_2x05_P2.54mm_Horizontal, symbol Connector_Generic:Conn_02x05_Odd_Even
- removed R10, R11, R13: 10K, Resistor_SMD:R_0603_1608Metric, symbol Device:R
- removed R12: 2.2K, Resistor_SMD:R_0603_1608Metric, symbol Device:R
- removed R2, R3: 560, Resistor_SMD:R_0603_1608Metric, symbol Device:R
- removed SW1: SW_Push, Button_Switch_THT:SW_Tactile_SPST_Angled_PTS645Vx39-2LFS, symbol Switch:SW_Push
Connections:
- net VDD3V3 is gone; now on net +3V3: U4.2 (VDD)
