File: rev.2-heat/esp23 i3 heat thermostat/filtered_button.kicad_sch (KiCad schematic)
At the start: 3 parts

Commit message: initial layout for UX
Parts:
- R18: renamed from R?; footprint (none) -> Resistor_SMD:R_0603_1608Metric
- gave numbers to parts that had none: 2
Changed lines of the file:
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@@
   (symbol (lib_id "power:+3.3V") (at 158.75 57.15 0)
     (in_bom yes) (on_board yes) (fields_autoplaced)
-    (property "Reference" "#PWR?" (id 0) (at 158.75 60.96 0)
+    (property "Reference" "#PWR047" (id 0) (at 158.75 60.96 0)
       (effects (font (size 1.27 1.27)) hide)
     )
@@
   (symbol (lib_id "Switch:SW_MEC_5E") (at 147.32 67.31 0)
     (in_bom yes) (on_board yes) (fields_autoplaced)
-    (property "Reference" "SW?" (id 0) (at 147.32 57.8825 0))
+    (property "Reference" "SW5" (id 0) (at 147.32 57.8825 0))
     (property "Value" "SW_MEC_5E" (id 1) (at 147.32 60.6576 0))
     (property "Footprint" "Button_Switch_THT:SW_TH_Tactile_Omron_B3F-10xx" (id 2) (at 147.32 59.69 0)
@@
   (symbol (lib_id "Device:C") (at 147.32 71.12 90)
     (in_bom yes) (on_board yes) (fields_autoplaced)
-    (property "Reference" "C?" (id 0) (at 147.32 64.9945 90))
+    (property "Reference" "C11" (id 0) (at 147.32 64.9945 90))
     (property "Value" "1nF" (id 1) (at 147.32 67.7696 90))
     (property "Footprint" "Capacitor_SMD:C_0603_1608Metric" (id 2) (at 151.13 70.1548 0)
@@
   (symbol (lib_id "Device:R") (at 158.75 60.96 0)
     (in_bom yes) (on_board yes) (fields_autoplaced)
-    (property "Reference" "R?" (id 0) (at 160.528 60.0515 0)
+    (property "Reference" "R18" (id 0) (at 160.528 60.0515 0)
       (effects (font (size 1.27 1.27)) (justify left))
     )
@@
       (effects (font (size 1.27 1.27)) (justify left))
     )
-    (property "Footprint" "" (id 2) (at 156.972 60.96 90)
+    (property "Footprint" "Resistor_SMD:R_0603_1608Metric" (id 2) (at 156.972 60.96 90)
       (effects (font (size 1.27 1.27)) hide)
     )
@@
   (symbol (lib_id "power:GND") (at 142.24 72.39 0)
     (in_bom yes) (on_board yes) (fields_autoplaced)
-    (property "Reference" "#PWR?" (id 0) (at 142.24 78.74 0)
+    (property "Reference" "#PWR046" (id 0) (at 142.24 78.74 0)
       (effects (font (size 1.27 1.27)) hide)
     )

Commit message: layout attempt 1
Parts:
- renumbered C11 to C8, R18 to R15, SW5 to SW2
Changed lines of the file:
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@@
   (symbol (lib_id "power:+3.3V") (at 158.75 57.15 0)
     (in_bom yes) (on_board yes) (fields_autoplaced)
-    (property "Reference" "#PWR047" (id 0) (at 158.75 60.96 0)
+    (property "Reference" "#PWR041" (id 0) (at 158.75 60.96 0)
       (effects (font (size 1.27 1.27)) hide)
     )
@@
   (symbol (lib_id "Switch:SW_MEC_5E") (at 147.32 67.31 0)
     (in_bom yes) (on_board yes) (fields_autoplaced)
-    (property "Reference" "SW5" (id 0) (at 147.32 57.8825 0))
+    (property "Reference" "SW2" (id 0) (at 147.32 57.8825 0))
     (property "Value" "SW_MEC_5E" (id 1) (at 147.32 60.6576 0))
     (property "Footprint" "Button_Switch_THT:SW_TH_Tactile_Omron_B3F-10xx" (id 2) (at 147.32 59.69 0)
@@
   (symbol (lib_id "Device:C") (at 147.32 71.12 90)
     (in_bom yes) (on_board yes) (fields_autoplaced)
-    (property "Reference" "C11" (id 0) (at 147.32 64.9945 90))
+    (property "Reference" "C8" (id 0) (at 147.32 64.9945 90))
     (property "Value" "1nF" (id 1) (at 147.32 67.7696 90))
     (property "Footprint" "Capacitor_SMD:C_0603_1608Metric" (id 2) (at 151.13 70.1548 0)
@@
   (symbol (lib_id "Device:R") (at 158.75 60.96 0)
     (in_bom yes) (on_board yes) (fields_autoplaced)
-    (property "Reference" "R18" (id 0) (at 160.528 60.0515 0)
+    (property "Reference" "R15" (id 0) (at 160.528 60.0515 0)
       (effects (font (size 1.27 1.27)) (justify left))
     )
@@
   (symbol (lib_id "power:GND") (at 142.24 72.39 0)
     (in_bom yes) (on_board yes) (fields_autoplaced)
-    (property "Reference" "#PWR046" (id 0) (at 142.24 78.74 0)
+    (property "Reference" "#PWR040" (id 0) (at 142.24 78.74 0)
       (effects (font (size 1.27 1.27)) hide)
     )
